File: AetherX_KiCad/AetherX_KiCad.kicad_pcb (KiCad board)
At the start: 2 copper layers, 125 x 72.5 mm, 36 parts, among them SW1 SW_Push, SW2 SW_Push, U1 STM32F401RETx, U2 DHT20, U3 MAX9814, U4 LM61, U5 SSD1306, U6 OPT101, Y1 8MHz

Commit message: PCB ordered, uploaded BOM and gerber files
Parts:
- added G***: LOGO, Random:star_wars_res, F.Cu at (210.2, 118.8)
- added G***: LOGO, Random:st_2, F.Cu at (173.5, 89.5)
- added MO1: MountingHole_4.3mm_M4, Mounting:MountingHole_4.3mm_M4, F.Cu at (102.0, 69.2)
- moved MO3 11.5 mm to (102.5, 129.2)
- moved MO2 2.55 mm to (221.5, 69.2)
- moved MO4 2.00 mm to (221.2, 128.5)
- renumbered MO3 to MO2, MO2 to MO3, MO1 to MO4
Routing:
- net Net-(U1-PH0): track 50.3 -> 53.1 mm
- net /ADC1_CH4: track 35.3 -> 36.3 mm
- net /Button1: track 53.2 -> 54.0 mm
- net Net-(U1-PC3): track 25.1 -> 24.6 mm
- net GND: vias 10 -> 5
Other:
- board size 125 x 72.5 mm -> 132.8 x 72.5 mm
- board text added: "OUT"
- board text added: "SCL"
- board text added: "SDA"
- board text added: "Screws: 4x M4"
- board text removed: "Use M4 screws to mount"
